Commit message: Refactor CAN communication: sync MIT send+receive, AK60-39 support, 7-motor config
- Remove async receiveLoop thread; replace with sendMITAndReceive (send + wait for response per motor)
- Add AK60-39 (motor 2) extended frame feedback decode (CAN ID 0x2902, int16 pos/current)
- Add AK60-39 disable via extended frame (CAN ID 0xF02, DLC=0)
- Add MITState.valid flag to prevent seeding hw_states from zero-initialized data
- Add kp_cmd/kd_cmd per-motor defaults in MotorParams presets
- Expand system to 7 motors: joint7 as gripper, separate gripper_controller
- Add mit_enable ROS topic for per-motor enable (0=all, 1-7=single)
- Add sendExt to CanBridge for 29-bit extended CAN frames
- Remove servo mode code, keep MIT only
- Add trajectory.py direct serial MIT tool with AK60-39 support

File: src/arm6dof/urdf/arm6dof.urdf (robot description, URDF)
Before this commit: robot arm6dof, 13 links, 12 joints
Links:
- added link joint7_link
Joints:
- added joint joint7: type continuous, parent jedziemy_dalej_V2_silnik_ak45-10-Kopiuj-v1, child joint7_link, origin xyz=0 0 0 rpy=0 0 0, axis 0 0 1

File: src/arm6dof_moveit_config
/config/arm6dof.ros2_control.xacro (robot description, xacro)
@@ -10,4 +10,5 @@
             <joint name="joint1">
                 <command_interface name="position"/>
+                <command_interface name="velocity"/>
                 <state_interface name="position">
                   <param name="initial_value">${initial_positions['joint1']}</param>
@@ -17,4 +18,5 @@
             <joint name="joint2">
                 <command_interface name="position"/>
+                <command_interface name="velocity"/>
                 <state_interface name="position">
                   <param name="initial_value">${initial_positions['joint2']}</param>
@@ -24,4 +26,5 @@
             <joint name="joint3">
                 <command_interface name="position"/>
+                <command_interface name="velocity"/>
                 <state_interface name="position">
                   <param name="initial_value">${initial_positions['joint3']}</param>
@@ -31,4 +34,5 @@
             <joint name="joint4">
                 <command_interface name="position"/>
+                <command_interface name="velocity"/>
                 <state_interface name="position">
                   <param name="initial_value">${initial_positions['joint4']}</param>
@@ -38,4 +42,5 @@
             <joint name="joint5">
                 <command_interface name="position"/>
+                <command_interface name="velocity"/>
                 <state_interface name="position">
                   <param name="initial_value">${initial_positions['joint5']}</param>
@@ -45,6 +50,15 @@
             <joint name="joint6">
                 <command_interface name="position"/>
+                <command_interface name="velocity"/>
                 <state_interface name="position">
                   <param name="initial_value">${initial_positions['joint6']}</param>
+                </state_interface>
+                <state_interface name="velocity"/>
+            </joint>
+            <joint name="joint7">
+                <command_interface name="position"/>
+                <command_interface name="velocity"/>
+                <state_interface name="position">
+                  <param name="initial_value">${initial_positions['joint7']}</param>
                 </state_interface>
                 <state_interface name="velocity"/>
